File: ssd1332_breakout/ssd1332_breakout.sch (KiCad schematic (older format))
At the start: 17 parts, among them P1 CONN_01X07, P2 CONN_01X27, U1 MC34063

Commit message: Started SSD1332 board
TODO:

* Check display header
* Pick smaller components
* Scan one of the OLED breakout PCBs and import outline from it
* Check about MC34063 layout guidelines
Parts:
- C1, C2, C3, C4, C5: footprint (none) -> Capacitors_SMD:C_0805_HandSoldering
- D1: footprint (none) -> Diodes_SMD:D_MiniMELF_Handsoldering
- L1: footprint (none) -> Choke_SMD:Choke_SMD_1206_Handsoldering
- P1: footprint (none) -> Pin_Headers:Pin_Header_Straight_1x07_Pitch2.54mm
- P2: footprint (none) -> footprints:FPC_27
- R1, R2, R3, R4, R5: footprint (none) -> Resistors_SMD:R_0805_HandSoldering
- U1: footprint (none) -> Housings_SOIC:SOIC-8_3.9x4.9mm_Pitch1.27mm
- W1, W2: footprint (none) -> Measurement_Points:Measurement_Point_Square-SMD-Pad_Small
Changed lines of the file:
@@
 LIBS:valves
 LIBS:mc34063
+LIBS:ssd1332_breakout-cache
 EELAYER 25 0
 EELAYER END
@@
 F 0 "P2" H 4600 5050 50  0000 C CNN
 F 1 "CONN_01X27" V 4700 3650 50  0000 C CNN
-F 2 "" H 4600 3650 50  0000 C CNN
+F 2 "footprints:FPC_27" H 4600 3650 50  0001 C CNN
 F 3 "" H 4600 3650 50  0000 C CNN
 	1    4600 3650
@@
 NoConn ~ 4400 4950
 $Comp
-L GND #PWR25
+L GND #PWR01
 U 1 1 58BBC39F
 P 4400 4850
-F 0 "#PWR25" H 4400 4600 50  0001 C CNN
+F 0 "#PWR01" H 4400 4600 50  0001 C CNN
 F 1 "GND" V 4400 4650 50  0000 C CNN
 F 2 "" H 4400 4850 50  0000 C CNN
@@
 $EndComp
 $Comp
-L GND #PWR15
+L GND #PWR02
 U 1 1 58BBC3CE
 P 4400 2450
-F 0 "#PWR15" H 4400 2200 50  0001 C CNN
+F 0 "#PWR02" H 4400 2200 50  0001 C CNN
 F 1 "GND" V 4400 2250 50  0000 C CNN
 F 2 "" H 4400 2450 50  0000 C CNN
@@
 $EndComp
 $Comp
-L VDD #PWR16
+L VDD #PWR03
 U 1 1 58BBC42C
 P 4400 2550
-F 0 "#PWR16" H 4400 2400 50  0001 C CNN
+F 0 "#PWR03" H 4400 2400 50  0001 C CNN
 F 1 "VDD" V 4400 2750 50  0000 C CNN
 F 2 "" H 4400 2550 50  0000 C CNN
@@
 $EndComp
 $Comp
-L VDD #PWR24
+L VDD #PWR04
 U 1 1 58BBC44E
 P 4400 4750
-F 0 "#PWR24" H 4400 4600 50  0001 C CNN
+F 0 "#PWR04" H 4400 4600 50  0001 C CNN
 F 1 "VDD" V 4400 4950 50  0000 C CNN
 F 2 "" H 4400 4750 50  0000 C CNN
@@
 $EndComp
 $Comp
-L VCC #PWR23
+L VCC #PWR05
 U 1 1 58BBC47E
 P 4400 4650
-F 0 "#PWR23" H 4400 4500 50  0001 C CNN
+F 0 "#PWR05" H 4400 4500 50  0001 C CNN
 F 1 "VCC" V 4400 4850 50  0000 C CNN
 F 2 "" H 4400 4650 50  0000 C CNN
@@
 $EndComp
 $Comp
-L VCC #PWR17
+L VCC #PWR06
 U 1 1 58BBC4A0
 P 4400 2650
-F 0 "#PWR17" H 4400 2500 50  0001 C CNN
+F 0 "#PWR06" H 4400 2500 50  0001 C CNN
 F 1 "VCC" V 4400 2850 50  0000 C CNN
 F 2 "" H 4400 2650 50  0000 C CNN
@@
 $EndComp
 $Comp
-L VCOM #PWR18
+L VCOM #PWR07
 U 1 1 58BBC4D3
 P 4400 2750
-F 0 "#PWR18" H 4400 2600 50  0001 C CNN
+F 0 "#PWR07" H 4400 2600 50  0001 C CNN
 F 1 "VCOM" V 4400 3000 50  0000 C CNN
 F 2 "" H 4400 2750 50  0000 C CNN
@@
 $EndComp
 $Comp
-L VCOM #PWR22
+L VCOM #PWR08
 U 1 1 58BBC51B
 P 4400 4550
-F 0 "#PWR22" H 4400 4400 50  0001 C CNN
+F 0 "#PWR08" H 4400 4400 50  0001 C CNN
 F 1 "VCOM" V 4400 4800 50  0000 C CNN
 F 2 "" H 4400 4550 50  0000 C CNN
@@
 $EndComp
 $Comp
-L VDD #PWR21
+L VDD #PWR09
 U 1 1 58BBC543
 P 4400 4450
-F 0 "#PWR21" H 4400 4300 50  0001 C CNN
+F 0 "#PWR09" H 4400 4300 50  0001 C CNN
 F 1 "VDD" V 4400 4650 50  0000 C CNN
 F 2 "" H 4400 4450 50  0000 C CNN
@@
 $EndComp
 $Comp
-L GND #PWR20
+L GND #PWR010
 U 1 1 58BBC565
 P 4400 4350
-F 0 "#PWR20" H 4400 4100 50  0001 C CNN
+F 0 "#PWR010" H 4400 4100 50  0001 C CNN
 F 1 "GND" V 4400 4150 50  0000 C CNN
 F 2 "" H 4400 4350 50  0000 C CNN
@@
 $EndComp
 $Comp
-L GND #PWR19
+L GND #PWR011
 U 1 1 58BBC573
 P 4400 4250
-F 0 "#PWR19" H 4400 4000 50  0001 C CNN
+F 0 "#PWR011" H 4400 4000 50  0001 C CNN
 F 1 "GND" V 4400 4050 50  0000 C CNN
 F 2 "" H 4400 4250 50  0000 C CNN
@@
 F 0 "R5" V 4200 4000 50  0000 C CNN
 F 1 "910K" V 4250 4150 50  0000 C CNN
-F 2 "" V 4180 4150 50  0000 C CNN
+F 2 "Resistors_SMD:R_0805_HandSoldering" V 4180 4150 50  0001 C CNN
 F 3 "" H 4250 4150 50  0000 C CNN
 	1    4250 4150
@@
 $EndComp
 $Comp
-L GND #PWR14
+L GND #PWR012
 U 1 1 58BBC5D5
 P 4100 4150
-F 0 "#PWR14" H 4100 3900 50  0001 C CNN
+F 0 "#PWR012" H 4100 3900 50  0001 C CNN
 F 1 "GND" V 4100 3950 50  0000 C CNN
 F 2 "" H 4100 4150 50  0000 C CNN
@@
 F 0 "R2" V 3500 3150 50  0000 C CNN
 F 1 "470" V 3400 3050 50  0000 C CNN
-F 2 "" V 3330 3050 50  0000 C CNN
+F 2 "Resistors_SMD:R_0805_HandSoldering" V 3330 3050 50  0001 C CNN
 F 3 "" H 3400 3050 50  0000 C CNN
 	1    3400 3050
@@
 $EndComp
 $Comp
-L VCC #PWR10
+L VCC #PWR013
 U 1 1 58BBC79F
 P 3550 3050
-F 0 "#PWR10" H 3550 2900 50  0001 C CNN
+F 0 "#PWR013" H 3550 2900 50  0001 C CNN
 F 1 "VCC" V 3550 3250 50  0000 C CNN
 F 2 "" H 3550 3050 50  0000 C CNN
@@
 $EndComp
 $Comp
-L VEE #PWR6
+L VEE #PWR014
 U 1 1 58BBC7DC
 P 3250 3050
-F 0 "#PWR6" H 3250 2900 50  0001 C CNN
+F 0 "#PWR014" H 3250 2900 50  0001 C CNN
 F 1 "VEE" V 3250 3250 50  0000 C CNN
 F 2 "" H 3250 3050 50  0000 C CNN
@@
 F 0 "C5" H 3875 2600 50  0000 L CNN
 F 1 "4.7uF" H 3875 2400 50  0000 L CNN
-F 2 "" H 3888 2350 50  0000 C CNN
+F 2 "Capacitors_SMD:C_0805_HandSoldering" H 3888 2350 50  0001 C CNN
 F 3 "" H 3850 2500 50  0000 C CNN
 	1    3850 2500
@@
 $EndComp
 $Comp
-L GND #PWR13
+L GND #PWR015
 U 1 1 58BBC8E3
 P 3850 2650
-F 0 "#PWR13" H 3850 2400 50  0001 C CNN
+F 0 "#PWR015" H 3850 2400 50  0001 C CNN
 F 1 "GND" H 4000 2550 50  0000 C CNN
 F 2 "" H 3850 2650 50  0000 C CNN
@@
 $EndComp
 $Comp
-L VCOM #PWR12
+L VCOM #PWR016
 U 1 1 58BBC941
 P 3850 2350
-F 0 "#PWR12" H 3850 2200 50  0001 C CNN
+F 0 "#PWR016" H 3850 2200 50  0001 C CNN
 F 1 "VCOM" H 4050 2450 50  0000 C CNN
 F 2 "" H 3850 2350 50  0000 C CNN
@@
 F 0 "C3" H 3475 2600 50  0000 L CNN
 F 1 "4.7uF" H 3475 2400 50  0000 L CNN
-F 2 "" H 3488 2350 50  0000 C CNN
+F 2 "Capacitors_SMD:C_0805_HandSoldering" H 3488 2350 50  0001 C CNN
 F 3 "" H 3450 2500 50  0000 C CNN
 	1    3450 2500
@@
 $EndComp
 $Comp
-L GND #PWR8
+L GND #PWR017
 U 1 1 58BBC9F9
 P 3450 2650
-F 0 "#PWR8" H 3450 2400 50  0001 C CNN
+F 0 "#PWR017" H 3450 2400 50  0001 C CNN
 F 1 "GND" H 3600 2550 50  0000 C CNN
 F 2 "" H 3450 2650 50  0000 C CNN
@@
 $EndComp
 $Comp
-L VDD #PWR7
+L VDD #PWR018
 U 1 1 58BBCA0B
 P 3450 2350
-F 0 "#PWR7" H 3450 2200 50  0001 C CNN
+F 0 "#PWR018" H 3450 2200 50  0001 C CNN
 F 1 "VDD" H 3600 2450 50  0000 C CNN
 F 2 "" H 3450 2350 50  0000 C CNN
@@
 F 0 "C2" H 3075 2600 50  0000 L CNN
 F 1 "4.7uF" H 3075 2400 50  0000 L CNN
-F 2 "" H 3088 2350 50  0000 C CNN
+F 2 "Capacitors_SMD:C_0805_HandSoldering" H 3088 2350 50  0001 C CNN
 F 3 "" H 3050 2500 50  0000 C CNN
 	1    3050 2500
@@
 $EndComp
 $Comp
-L GND #PWR5
+L GND #PWR019
 U 1 1 58BBCA70
 P 3050 2650
-F 0 "#PWR5" H 3050 2400 50  0001 C CNN
+F 0 "#PWR019" H 3050 2400 50  0001 C CNN
 F 1 "GND" H 3200 2550 50  0000 C CNN
 F 2 "" H 3050 2650 50  0000 C CNN
@@
 $EndComp
 $Comp
-L VCC #PWR4
+L VCC #PWR020
 U 1 1 58BBCA91
 P 3050 2350
-F 0 "#PWR4" H 3050 2200 50  0001 C CNN
+F 0 "#PWR020" H 3050 2200 50  0001 C CNN
 F 1 "VCC" H 3200 2450 50  0000 C CNN
 F 2 "" H 3050 2350 50  0000 C CNN
@@
 F 0 "P1" H 2450 2950 50  0000 C CNN
 F 1 "CONN_01X07" V 2550 2550 50  0000 C CNN
-F 2 "" H 2450 2550 50  0000 C CNN
+F 2 "Pin_Headers:Pin_Header_Straight_1x07_Pitch2.54mm" H 2450 2550 50  0001 C CNN
 F 3 "" H 2450 2550 50  0000 C CNN
 	1    2450 2550
@@
 $EndComp
 $Comp
-L GND #PWR3
+L GND #PWR021
 U 1 1 58BBCBED
 P 2650 2850
-F 0 "#PWR3" H 2650 2600 50  0001 C CNN
+F 0 "#PWR021" H 2650 2600 50  0001 C CNN
 F 1 "GND" V 2650 2650 50  0000 C CNN
 F 2 "" H 2650 2850 50  0000 C CNN
@@
 $EndComp
 $Comp
-L VEE #PWR2
+L VEE #PWR022
 U 1 1 58BBCC0D
 P 2650 2750
-F 0 "#PWR2" H 2650 2600 50  0001 C CNN
+F 0 "#PWR022" H 2650 2600 50  0001 C CNN
 F 1 "VEE" V 2650 2950 50  0000 C CNN
 F 2 "" H 2650 2750 50  0000 C CNN
@@
 F 0 "U1" H 2800 3450 60  0000 C CNN
 F 1 "MC34063" H 2900 4050 60  0000 C CNN
-F 2 "" H 2950 3800 60  0001 C CNN
+F 2 "Housings_SOIC:SOIC-8_3.9x4.9mm_Pitch1.27mm" H 2950 3800 60  0001 C CNN
 F 3 "" H 2950 3800 60  0001 C CNN
 	1    2950 3750
@@
 $EndComp
 $Comp
-L GND #PWR1
+L GND #PWR023
 U 1 1 58BBD1BC
 P 2200 3900
-F 0 "#PWR1" H 2200 3650 50  0001 C CNN
+F 0 "#PWR023" H 2200 3650 50  0001 C CNN
 F 1 "GND" H 2300 3800 50  0000 C CNN
 F 2 "" H 2200 3900 50  0000 C CNN
@@
 F 0 "W1" V 3600 4000 50  0000 C CNN
 F 1 "VIN" V 3500 4000 50  0000 C CNN
-F 2 "" H 3750 3800 50  0000 C CNN
+F 2 "Measurement_Points:Measurement_Point_Square-SMD-Pad_Small" H 3750 3800 50  0001 C CNN
 F 3 "" H 3750 3800 50  0000 C CNN
 	1    3550 3800
@@
 F 0 "R4" V 3600 3900 50  0000 C CNN
 F 1 "1.2K" V 3500 3900 50  0000 C CNN
-F 2 "" V 3430 3900 50  0000 C CNN
+F 2 "Resistors_SMD:R_0805_HandSoldering" V 3430 3900 50  0001 C CNN
 F 3 "" H 3500 3900 50  0000 C CNN
 	1    3500 3900
@@
 F 0 "R3" V 3600 3600 50  0000 C CNN
 F 1 "033" V 3500 3600 50  0000 C CNN
-F 2 "" V 3430 3600 50  0000 C CNN
+F 2 "Resistors_SMD:R_0805_HandSoldering" V 3430 3600 50  0001 C CNN
 F 3 "" H 3500 3600 50  0000 C CNN
 	1    3500 3600
@@
 $EndComp
 $Comp
-L GND #PWR11
+L GND #PWR024
 U 1 1 58BBDB9B
 P 3700 3900
-F 0 "#PWR11" H 3700 3650 50  0001 C CNN
+F 0 "#PWR024" H 3700 3650 50  0001 C CNN
 F 1 "GND" H 3850 3850 50  0000 C CNN
 F 2 "" H 3700 3900 50  0000 C CNN
@@
 F 0 "D1" H 2500 3600 50  0000 C CNN
 F 1 "1N5819" H 2350 3550 50  0000 C CNN
-F 2 "" H 2350 3650 50  0000 C CNN
+F 2 "Diodes_SMD:D_MiniMELF_Handsoldering" H 2350 3650 50  0001 C CNN
 F 3 "" H 2350 3650 50  0000 C CNN
 	1    2350 3650
@@
 F 0 "W2" V 3600 4500 50  0000 C CNN
 F 1 "VOUT" V 3500 4550 50  0000 C CNN
-F 2 "" H 3750 4300 50  0000 C CNN
+F 2 "Measurement_Points:Measurement_Point_Square-SMD-Pad_Small" H 3750 4300 50  0001 C CNN
 F 3 "" H 3750 4300 50  0000 C CNN
 	1    3550 4300
@@
 F 0 "C1" V 2400 3850 50  0000 L CNN
 F 1 "470P" V 2300 3850 50  0000 L CNN
-F 2 "" H 2388 3650 50  0000 C CNN
+F 2 "Capacitors_SMD:C_0805_HandSoldering" H 2388 3650 50  0001 C CNN
 F 3 "" H 2350 3800 50  0000 C CNN
 	1    2350 3800
@@
 F 0 "C4" H 3350 4450 50  0000 L CNN
 F 1 "470" H 3250 4650 50  0000 L CNN
-F 2 "" H 3488 4400 50  0000 C CNN
+F 2 "Capacitors_SMD:C_0805_HandSoldering" H 3488 4400 50  0001 C CNN
 F 3 "" H 3450 4550 50  0000 C CNN
 	1    3450 4550
@@
 $EndComp
 $Comp
-L GND #PWR9
+L GND #PWR025
 U 1 1 58BBE9AD
 P 3450 4700
-F 0 "#PWR9" H 3450 4450 50  0001 C CNN
+F 0 "#PWR025" H 3450 4450 50  0001 C CNN
 F 1 "GND" H 3600 4650 50  0000 C CNN
 F 2 "" H 3450 4700 50  0000 C CNN
@@
 F 0 "L1" V 3150 4300 50  0000 L CNN
 F 1 "220uH" V 3050 4250 50  0000 L CNN
-F 2 "" H 3100 4300 50  0000 C CNN
+F 2 "Choke_SMD:Choke_SMD_1206_Handsoldering" H 3100 4300 50  0001 C CNN
 F 3 "" H 3100 4300 50  0000 C CNN
 	1    3100 4300
@@
 F 0 "R1" V 3450 4150 50  0000 C CNN
 F 1 "45K" V 3350 4150 50  0000 C CNN
-F 2 "" V 3280 4150 50  0000 C CNN
+F 2 "Resistors_SMD:R_0805_HandSoldering" V 3280 4150 50  0001 C CNN
 F 3 "" H 3350 4150 50  0000 C CNN
 	1    3350 4150
