File: keypad_pcb/keypad_prototype.kicad_pcb (KiCad board)
At the start: 2 copper layers, 40 x 60 mm, 32 parts

Commit message: Silkscreen additions for keypad board
-Notes on soldering
-Tips for soldering
-Pin names
Connections:
- ? pad 1: Net-(C2-Pad1) -> (no net)
- ? pad 10: Net-(N*1-Pad2) -> (no net)
- ? pad 11: Net-(C5-Pad2) -> (no net)
- ? pad 2: Net-(C4-Pad1) -> (no net)
- ? pad 3: Net-(C1-Pad1) -> (no net)
- ? pad 4: Net-(C3-Pad1) -> (no net)
- ? pad 5: Net-(C5-Pad1) -> (no net)
- ? pad 6: Net-(C1-Pad2) -> (no net)
- ? pad 7: Net-(GREEN1-Pad2) -> (no net)
- ? pad 8: Net-(C3-Pad2) -> (no net)
- ? pad 9: Net-(N2-Pad2) -> (no net)
- C1 pad 1: Net-(C1-Pad1) -> /ROW3
- C1 pad 2: Net-(C1-Pad2) -> /COL1
- C2 pad 1: Net-(C2-Pad1) -> /ROW1
- C2 pad 2: Net-(C1-Pad2) -> /COL1
- C3 pad 1: Net-(C3-Pad1) -> /ROW4
- C3 pad 2: Net-(C3-Pad2) -> /COL3
- C4 pad 1: Net-(C4-Pad1) -> /ROW2
- C4 pad 2: Net-(C3-Pad2) -> /COL3
- C5 pad 1: Net-(C5-Pad1) -> /ROW5
- C5 pad 2: Net-(C5-Pad2) -> /COL6
- C6 pad 1: Net-(C4-Pad1) -> /ROW2
- C6 pad 2: Net-(C5-Pad2) -> /COL6
- DOWN1 pad 1: Net-(C1-Pad1) -> /ROW3
- DOWN1 pad 2: Net-(C3-Pad2) -> /COL3
- GREEN1 pad 1: Net-(C5-Pad1) -> /ROW5
- GREEN1 pad 2: Net-(GREEN1-Pad2) -> /COL2
- LEFT1 pad 1: Net-(C3-Pad1) -> /ROW4
- LEFT1 pad 2: Net-(GREEN1-Pad2) -> /COL2
- N#1 pad 1: Net-(C1-Pad1) -> /ROW3
- N#1 pad 2: Net-(C5-Pad2) -> /COL6
- N*1 pad 1: Net-(C3-Pad1) -> /ROW4
- N*1 pad 2: Net-(N*1-Pad2) -> /COL5
- N0 pad 1: Net-(C3-Pad1) -> /ROW4
- N0 pad 2: Net-(C5-Pad2) -> /COL6
- N1 pad 1: Net-(C5-Pad1) -> /ROW5
- N1 pad 2: Net-(C3-Pad2) -> /COL3
- N2 pad 1: Net-(C1-Pad1) -> /ROW3
- N2 pad 2: Net-(N2-Pad2) -> /COL4
- N3 pad 1: Net-(C2-Pad1) -> /ROW1
- N3 pad 2: Net-(C3-Pad2) -> /COL3
- N4 pad 1: Net-(C5-Pad1) -> /ROW5
- N4 pad 2: Net-(N2-Pad2) -> /COL4
- N5 pad 1: Net-(C4-Pad1) -> /ROW2
- N5 pad 2: Net-(N2-Pad2) -> /COL4
- N6 pad 1: Net-(C2-Pad1) -> /ROW1
- N6 pad 2: Net-(N2-Pad2) -> /COL4
- N7 pad 1: Net-(C1-Pad1) -> /ROW3
- N7 pad 2: Net-(N*1-Pad2) -> /COL5
- N8 pad 1: Net-(C3-Pad1) -> /ROW4
- N8 pad 2: Net-(N2-Pad2) -> /COL4
- N9 pad 1: Net-(C4-Pad1) -> /ROW2
- N9 pad 2: Net-(N*1-Pad2) -> /COL5
- OK1 pad 1: Net-(C1-Pad1) -> /ROW3
- OK1 pad 2: Net-(GREEN1-Pad2) -> /COL2
- OPTION1 pad 1: Net-(C5-Pad1) -> /ROW5
- OPTION1 pad 2: Net-(N*1-Pad2) -> /COL5
- PHOTO1 pad 1: Net-(C2-Pad1) -> /ROW1
- PHOTO1 pad 2: Net-(N*1-Pad2) -> /COL5
- PHOTO2 pad 1: Net-(C2-Pad1) -> /ROW1
- PHOTO2 pad 2: Net-(C5-Pad2) -> /COL6
- RED1 pad 1: Net-(C2-Pad1) -> /ROW1
- RED1 pad 2: Net-(GREEN1-Pad2) -> /COL2
- RIGHT1 pad 1: Net-(C4-Pad1) -> /ROW2
- RIGHT1 pad 2: Net-(GREEN1-Pad2) -> /COL2
- UP1 pad 1: Net-(C4-Pad1) -> /ROW2
- UP1 pad 2: Net-(C1-Pad2) -> /COL1
- VOL_DOWN1 pad 1: Net-(C5-Pad1) -> /ROW5
- VOL_DOWN1 pad 2: Net-(C1-Pad2) -> /COL1
- VOL_UP1 pad 1: Net-(C3-Pad1) -> /ROW4
- VOL_UP1 pad 2: Net-(C1-Pad2) -> /COL1
Routing:
- net Net-(C1-Pad1): track 121.8 -> 0.00 mm, vias 9 -> 0
- net /ROW3: track 0.00 -> 121.8 mm, vias 0 -> 9
- net Net-(C5-Pad1): track 120.8 -> 0.00 mm, vias 7 -> 0
- net /ROW5: track 0.00 -> 120.8 mm, vias 0 -> 7
- net Net-(C4-Pad1): track 106.1 -> 0.00 mm, vias 8 -> 0
- net /ROW2: track 0.00 -> 106.1 mm, vias 0 -> 8
- net Net-(C3-Pad1): track 104.6 -> 0.00 mm, vias 8 -> 0
- net /ROW4: track 0.00 -> 104.6 mm, vias 0 -> 8
- net Net-(C1-Pad2): track 86.2 -> 0.00 mm, vias 3 -> 0
- net /COL1: track 0.00 -> 86.2 mm, vias 0 -> 3
- net Net-(C2-Pad1): track 81.7 -> 0.00 mm, vias 5 -> 0
- net /ROW1: track 0.00 -> 81.7 mm, vias 0 -> 5
- net Net-(N*1-Pad2): track 79.5 -> 0.00 mm, vias 5 -> 0
- net /COL5: track 0.00 -> 79.5 mm, vias 0 -> 5
- net Net-(N2-Pad2): track 79.1 -> 0.00 mm, vias 6 -> 0
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Other:
- board text added: "1. Solder 4-pin buttons in the center row 2. Solder first and third rows of 4-pin buttons 3. Solder 2-pin buttons 4. Flip the board, solder side buttons (you can tack them on with superglue first) 5. Solder the headers on, facing downwards"
- board text added: "BL- BL+"
- board text added: "C1 C2 C3"
- board text added: "C4 C5 C6"
- board text added: "GPIO"
- board text added: "If you're soldering SMD parts yourself, this might be the board to work on first. Solder one pad of the button on, adjust the button, solder the other pads, repeat."
- board text added: "R5 R4 R3 R2 R1"
- board text added: "VCC SDA SCL GND"
- board text removed: "Sorry, this side is not symmetric. The front side is much prettier, go look at it instead!"
