File: keypad_pcb/keypad_prototype.kicad_pcb (KiCad board)
At the start: 2 copper layers, 40 x 60 mm, 32 parts

Commit message: Bumping the revision
Other:
- board text added: "ZeroPhone Delta"
- board text removed: "ZeroPhone Gamma"
Changed lines of the file:
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@@
     (effects (font (size 1.5 1.5) (thickness 0.3)) (justify mirror))
   )
-  (gr_text "ZeroPhone\nGamma" (at 151.257 146.177 270) (layer F.SilkS)
+  (gr_text "ZeroPhone\nDelta" (at 151.257 146.177 270) (layer F.SilkS)
     (effects (font (size 1.5 1.5) (thickness 0.3)))
   )
