File: keypad_pcb/keypad_pcb.sch (KiCad schematic (older format))
At the start: 31 parts, among them U1 KEYPAD_OVERLAY

Commit message: Started KiCad 5 migration
Opened each schematic, "rescued" symbols, then saved the files. No .kicad_pcb file changes so far.
Parts:
- C1, C2, C3, C4, C5, C6, DOWN1, GREEN1, LEFT1, N#1, N*1, N0, N1, N2, N3, N4, N5, N6, N7, N8, N9, OK1, OPTION1, PHOTO1, PHOTO2, RED1, RIGHT1, UP1, VOL_DOWN1, VOL_UP1: symbol AB2_SWITCH_MOMENTARY -> keypad_pcb-rescue:AB2_SWITCH_MOMENTARY
- U1: symbol KEYPAD_OVERLAY -> keypad_overlay:KEYPAD_OVERLAY
Changed lines of the file:
@@
-EESchema Schematic File Version 2
-LIBS:power
-LIBS:device
-LIBS:transistors
-LIBS:conn
-LIBS:linear
-LIBS:regul
-LIBS:74xx
-LIBS:cmos4000
-LIBS:adc-dac
-LIBS:memory
-LIBS:xilinx
-LIBS:microcontrollers
-LIBS:dsp
-LIBS:microchip
-LIBS:analog_switches
-LIBS:motorola
-LIBS:texas
-LIBS:intel
-LIBS:audio
-LIBS:interface
-LIBS:digital-audio
-LIBS:philips
-LIBS:display
-LIBS:cypress
-LIBS:siliconi
-LIBS:opto
-LIBS:atmel
-LIBS:contrib
-LIBS:valves
-LIBS:keypad_overlay
-LIBS:keypad_prototype-cache
-EELAYER 25 0
+EESchema Schematic File Version 4
+LIBS:keypad_pcb-cache
+EELAYER 26 0
 EELAYER END
 $Descr A4 11693 8268
@@
 $EndDescr
 $Comp
-L AB2_SWITCH_MOMENTARY VOL_DOWN1
+L keypad_pcb-rescue:AB2_SWITCH_MOMENTARY VOL_DOWN1
 U 1 1 58471E29
 P 2650 3500
@@
 $EndComp
 $Comp
-L AB2_SWITCH_MOMENTARY VOL_UP1
+L keypad_pcb-rescue:AB2_SWITCH_MOMENTARY VOL_UP1
 U 1 1 58471F6E
 P 3200 3500
@@
 $EndComp
 $Comp
-L AB2_SWITCH_MOMENTARY C1
+L keypad_pcb-rescue:AB2_SWITCH_MOMENTARY C1
 U 1 1 58471F97
 P 3750 3500
@@
 $EndComp
 $Comp
-L AB2_SWITCH_MOMENTARY UP1
+L keypad_pcb-rescue:AB2_SWITCH_MOMENTARY UP1
 U 1 1 58471FC1
 P 4300 3500
@@
 $EndComp
 $Comp
-L AB2_SWITCH_MOMENTARY C2
+L keypad_pcb-rescue:AB2_SWITCH_MOMENTARY C2
 U 1 1 58471FF2
 P 4850 3500
@@
 $EndComp
 $Comp
-L AB2_SWITCH_MOMENTARY GREEN1
+L keypad_pcb-rescue:AB2_SWITCH_MOMENTARY GREEN1
 U 1 1 584722B3
 P 2650 3850
@@
 $EndComp
 $Comp
-L AB2_SWITCH_MOMENTARY LEFT1
+L keypad_pcb-rescue:AB2_SWITCH_MOMENTARY LEFT1
 U 1 1 584722B9
 P 3200 3850
@@
 $EndComp
 $Comp
-L AB2_SWITCH_MOMENTARY OK1
+L keypad_pcb-rescue:AB2_SWITCH_MOMENTARY OK1
 U 1 1 584722BF
 P 3750 3850
@@
 $EndComp
 $Comp
-L AB2_SWITCH_MOMENTARY RIGHT1
+L keypad_pcb-rescue:AB2_SWITCH_MOMENTARY RIGHT1
 U 1 1 584722C5
 P 4300 3850
@@
 $EndComp
 $Comp
-L AB2_SWITCH_MOMENTARY RED1
+L keypad_pcb-rescue:AB2_SWITCH_MOMENTARY RED1
 U 1 1 584722CB
 P 4850 3850
@@
 $EndComp
 $Comp
-L AB2_SWITCH_MOMENTARY N1
+L keypad_pcb-rescue:AB2_SWITCH_MOMENTARY N1
 U 1 1 5847235A
 P 2650 4200
@@
 $EndComp
 $Comp
-L AB2_SWITCH_MOMENTARY C3
+L keypad_pcb-rescue:AB2_SWITCH_MOMENTARY C3
 U 1 1 58472360
 P 3200 4200
@@
 $EndComp
 $Comp
-L AB2_SWITCH_MOMENTARY DOWN1
+L keypad_pcb-rescue:AB2_SWITCH_MOMENTARY DOWN1
 U 1 1 58472366
 P 3750 4200
@@
 $EndComp
 $Comp
-L AB2_SWITCH_MOMENTARY C4
+L keypad_pcb-rescue:AB2_SWITCH_MOMENTARY C4
 U 1 1 5847236C
 P 4300 4200
@@
 $EndComp
 $Comp
-L AB2_SWITCH_MOMENTARY N3
+L keypad_pcb-rescue:AB2_SWITCH_MOMENTARY N3
 U 1 1 58472372
 P 4850 4200
@@
 $EndComp
 $Comp
-L AB2_SWITCH_MOMENTARY N4
+L keypad_pcb-rescue:AB2_SWITCH_MOMENTARY N4
 U 1 1 584724F1
 P 2650 4500
@@
 $EndComp
 $Comp
-L AB2_SWITCH_MOMENTARY N8
+L keypad_pcb-rescue:AB2_SWITCH_MOMENTARY N8
 U 1 1 584724F7
 P 3200 4500
@@
 $EndComp
 $Comp
-L AB2_SWITCH_MOMENTARY N2
+L keypad_pcb-rescue:AB2_SWITCH_MOMENTARY N2
 U 1 1 584724FD
 P 3750 4500
@@
 $EndComp
 $Comp
-L AB2_SWITCH_MOMENTARY N5
+L keypad_pcb-rescue:AB2_SWITCH_MOMENTARY N5
 U 1 1 58472503
 P 4300 4500
@@
 $EndComp
 $Comp
-L AB2_SWITCH_MOMENTARY N6
+L keypad_pcb-rescue:AB2_SWITCH_MOMENTARY N6
 U 1 1 58472509
 P 4850 4500
@@
 $EndComp
 $Comp
-L AB2_SWITCH_MOMENTARY OPTION1
+L keypad_pcb-rescue:AB2_SWITCH_MOMENTARY OPTION1
 U 1 1 5847250F
 P 2650 4850
@@
 $EndComp
 $Comp
-L AB2_SWITCH_MOMENTARY N*1
+L keypad_pcb-rescue:AB2_SWITCH_MOMENTARY N*1
 U 1 1 58472515
 P 3200 4850
@@
 $EndComp
 $Comp
-L AB2_SWITCH_MOMENTARY N7
+L keypad_pcb-rescue:AB2_SWITCH_MOMENTARY N7
 U 1 1 5847251B
 P 3750 4850
@@
 $EndComp
 $Comp
-L AB2_SWITCH_MOMENTARY N9
+L keypad_pcb-rescue:AB2_SWITCH_MOMENTARY N9
 U 1 1 58472521
 P 4300 4850
@@
 $EndComp
 $Comp
-L AB2_SWITCH_MOMENTARY PHOTO1
+L keypad_pcb-rescue:AB2_SWITCH_MOMENTARY PHOTO1
 U 1 1 58472527
 P 4850 4850
@@
 $EndComp
 $Comp
-L AB2_SWITCH_MOMENTARY C5
+L keypad_pcb-rescue:AB2_SWITCH_MOMENTARY C5
 U 1 1 5847252D
 P 2650 5200
@@
 $EndComp
 $Comp
-L AB2_SWITCH_MOMENTARY N0
+L keypad_pcb-rescue:AB2_SWITCH_MOMENTARY N0
 U 1 1 58472533
 P 3200 5200
@@
 $EndComp
 $Comp
-L AB2_SWITCH_MOMENTARY N#1
+L keypad_pcb-rescue:AB2_SWITCH_MOMENTARY N#1
 U 1 1 58472539
 P 3750 5200
@@
 $EndComp
 $Comp
-L AB2_SWITCH_MOMENTARY C6
+L keypad_pcb-rescue:AB2_SWITCH_MOMENTARY C6
 U 1 1 5847253F
 P 4300 5200
@@
 $EndComp
 $Comp
-L AB2_SWITCH_MOMENTARY PHOTO2
+L keypad_pcb-rescue:AB2_SWITCH_MOMENTARY PHOTO2
 U 1 1 58472545
 P 4850 5200
@@
 Connection ~ 2500 4850
 Wire Wire Line
-	3050 3300 3050 5200
+	3050 3300 3050 3500
 Connection ~ 3050 3850
 Connection ~ 3050 4200
@@
 Connection ~ 3050 4850
 Wire Wire Line
-	3600 3200 3600 5200
+	3600 3200 3600 3500
 Connection ~ 3600 3850
 Connection ~ 3600 4200
@@
 Connection ~ 3600 4850
 Wire Wire Line
-	4150 3100 4150 5200
+	4150 3100 4150 3500
 Connection ~ 4150 4850
 Connection ~ 4150 4500
@@
 Connection ~ 4150 3850
 Wire Wire Line
-	4700 3000 4700 5200
+	4700 3000 4700 3500
 Connection ~ 4700 4850
 Connection ~ 4700 4500
@@
 	2800 3500 2800 3600
 Wire Wire Line
-	2800 3600 5600 3600
+	2800 3600 3350 3600
 Connection ~ 3350 3600
 Connection ~ 3900 3600
@@
 	2800 3850 2800 3950
 Wire Wire Line
-	2800 3950 5700 3950
+	2800 3950 3350 3950
 Wire Wire Line
 	5000 3950 5000 3850
@@
 	2800 4200 2800 4300
 Wire Wire Line
-	2800 4300 5800 4300
+	2800 4300 3350 4300
 Wire Wire Line
 	5000 4300 5000 4200
@@
 	2800 4500 2800 4600
 Wire Wire Line
-	2800 4600 5900 4600
+	2800 4600 3350 4600
 Wire Wire Line
 	5000 4600 5000 4500
@@
 	2800 4850 2800 4950
 Wire Wire Line
-	2800 4950 6000 4950
+	2800 4950 3350 4950
 Wire Wire Line
 	5000 4950 5000 4850
@@
 	2800 5200 2800 5300
 Wire Wire Line
-	2800 5300 6100 5300
+	2800 5300 3350 5300
 Wire Wire Line
 	5000 5300 5000 5200
@@
 	3350 3600 3350 3500
 Wire Wire Line
-	2500 2300 2500 5200
+	2500 2300 2500 3500
 Wire Wire Line
 	2700 1900 3050 1900
@@
 NoConn ~ 3050 2550
 $Comp
-L KEYPAD_OVERLAY U1
+L keypad_overlay:KEYPAD_OVERLAY U1
 U 1 1 58866251
 P 3850 2100
@@
 Text Label 2800 2300 0    60   ~ 0
 ROW5
+Wire Wire Line
+	2500 3850 2500 4200
+Wire Wire Line
+	2500 4200 2500 4500
+Wire Wire Line
+	2500 4500 2500 4850
+Wire Wire Line
+	2500 4850 2500 5200
+Wire Wire Line
+	3050 3850 3050 4200
+Wire Wire Line
+	3050 4200 3050 4500
+Wire Wire Line
+	3050 4500 3050 4850
+Wire Wire Line
+	3050 4850 3050 5200
+Wire Wire Line
+	3600 3850 3600 4200
+Wire Wire Line
+	3600 4200 3600 4500
+Wire Wire Line
+	3600 4500 3600 4850
+Wire Wire Line
+	3600 4850 3600 5200
+Wire Wire Line
+	4150 4850 4150 5200
+Wire Wire Line
+	4150 4500 4150 4850
+Wire Wire Line
+	4150 4200 4150 4500
+Wire Wire Line
+	4150 3850 4150 4200
+Wire Wire Line
+	4700 4850 4700 5200
+Wire Wire Line
+	4700 4500 4700 4850
+Wire Wire Line
+	4700 4200 4700 4500
+Wire Wire Line
+	4700 3850 4700 4200
+Wire Wire Line
+	3350 3600 3900 3600
+Wire Wire Line
+	3900 3600 4450 3600
+Wire Wire Line
+	4450 3600 5000 3600
+Wire Wire Line
+	4450 3950 5000 3950
+Wire Wire Line
+	3900 3950 4450 3950
+Wire Wire Line
+	3350 3950 3900 3950
+Wire Wire Line
+	3350 4300 3900 4300
+Wire Wire Line
+	3350 4600 3900 4600
+Wire Wire Line
+	3350 4950 3900 4950
+Wire Wire Line
+	3350 5300 3900 5300
+Wire Wire Line
+	3900 5300 4450 5300
+Wire Wire Line
+	3900 4950 4450 4950
+Wire Wire Line
+	3900 4600 4450 4600
+Wire Wire Line
+	3900 4300 4450 4300
+Wire Wire Line
+	4450 4300 5000 4300
+Wire Wire Line
+	4450 4600 5000 4600
+Wire Wire Line
+	4450 4950 5000 4950
+Wire Wire Line
+	4450 5300 5000 5300
+Wire Wire Line
+	2500 3500 2500 3850
+Wire Wire Line
+	5000 5300 6100 5300
+Wire Wire Line
+	5000 4950 6000 4950
+Wire Wire Line
+	5000 4600 5900 4600
+Wire Wire Line
+	5000 4300 5800 4300
+Wire Wire Line
+	5000 3950 5700 3950
+Wire Wire Line
+	5000 3600 5600 3600
+Wire Wire Line
+	3050 3500 3050 3850
+Wire Wire Line
+	3600 3500 3600 3850
+Wire Wire Line
+	4150 3500 4150 3850
+Wire Wire Line
+	4700 3500 4700 3850
 $EndSCHEMATC
