File: 18650_pcb/18650_pcb.kicad_pcb (KiCad board)
At the start: 2 copper layers, 40 x 88 mm, 5 parts, among them P1 CONN_01X02

Commit message: Revision label updates, origin points
Other:
- board text added: "18650 PCB ZeroPhone Delta-B"
- board text removed: "18650 PCB ZeroPhone Delta"
Changed lines of the file:
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@@
   )
   (setup
-    (last_trace_width 3)
+    (last_trace_width 0.25)
     (user_trace_width 3)
     (trace_clearance 0.2)
@@
     (effects (font (size 3 3) (thickness 0.6)))
   )
-  (gr_text "18650 PCB\nZeroPhone Delta" (at 39.54702 30.49724) (layer B.SilkS)
+  (gr_text "18650 PCB\nZeroPhone Delta-B" (at 39.54702 30.49724) (layer B.SilkS)
     (effects (font (size 2 2) (thickness 0.4)) (justify mirror))
   )
@@
     (polygon
       (pts
-        (xy 19.86202 45.73724) (xy 26.08502 45.73724) (xy 26.08502 48.78524) (xy 19.86202 48.78524)
+        (xy 19.69902 45.75724) (xy 23.19902 45.75724) (xy 23.19902 48.75724) (xy 19.69902 48.75724)
       )
     )
@@
     (polygon
       (pts
-        (xy 19.73502 42.18124) (xy 26.08502 42.18124) (xy 26.08502 45.35624) (xy 19.73502 45.35624)
+        (xy 19.73502 42.18124) (xy 23.19902 42.15724) (xy 23.19902 45.35724) (xy 19.73502 45.35624)
       )
     )
