File: 6p_separator/6p_separator.sch (KiCad schematic (older format))
At the start: 1 part, among them J1 Conn_01x06

Commit message: Started KiCad 5 migration
Opened each schematic, "rescued" symbols, then saved the files. No .kicad_pcb file changes so far.
Parts:
- J1: symbol Conn_01x06 -> 6p_separator-rescue:Conn_01x06
Changed lines of the file:
@@
-EESchema Schematic File Version 2
-LIBS:power
-LIBS:device
-LIBS:switches
-LIBS:relays
-LIBS:motors
-LIBS:transistors
-LIBS:conn
-LIBS:linear
-LIBS:regul
-LIBS:74xx
-LIBS:cmos4000
-LIBS:adc-dac
-LIBS:memory
-LIBS:xilinx
-LIBS:microcontrollers
-LIBS:dsp
-LIBS:microchip
-LIBS:analog_switches
-LIBS:motorola
-LIBS:texas
-LIBS:intel
-LIBS:audio
-LIBS:interface
-LIBS:digital-audio
-LIBS:philips
-LIBS:display
-LIBS:cypress
-LIBS:siliconi
-LIBS:opto
-LIBS:atmel
-LIBS:contrib
-LIBS:valves
+EESchema Schematic File Version 4
 LIBS:6p_separator-cache
-EELAYER 25 0
+EELAYER 26 0
 EELAYER END
 $Descr A4 11693 8268
@@
 $EndDescr
 $Comp
-L Conn_01x06 J1
+L 6p_separator-rescue:Conn_01x06 J1
 U 1 1 5A86415A
 P 3750 3150
