File: back_pcb/back_pcb.sch (KiCad schematic (older format))
At the start: 118 parts, among them J1 Conn_01x12, P2 EXPANSION_BOTTOM, P3 EXPANSION_TOP, P4 AUDIO_CONN, P6 ATMEGA_HEADER, P7 EXPANSION_BOTTOM2, P8 JST, P9 USB_A, Q1 IRLML6401, Q2 IRLML6401, Q3 Q_PNP_BEC, Q4 IRLML6401, Q5 IRLML6401, Q6 IRLML6401, Q7 BC547, SW1 SW_PUSH, SW2 SW_PUSH, U1 PI ZERO, U2 SIM800_BREAKOUT, U3 MCP23017, U4 TP4056_BREAKOUT, U5 24C32, U6 DC_DC_BREAKOUT, U7 74LS125, U8 LM339

Commit message: Started KiCad 5 migration
Opened each schematic, "rescued" symbols, then saved the files. No .kicad_pcb file changes so far.
Parts:
- C1, C10, C11, C12, C13, C14, C15, C16, C17, C18, C19, C2, C20, C21, C22, C24, C25, C4, C5, C6, C7, C8, C9: symbol C_Small -> back_pcb-rescue:C_Small
- D1, D2, D6, D7: symbol D_Small -> back_pcb-rescue:D_Small
- D3: symbol Led_RGB_CA -> back_pcb-rescue:Led_RGB_CA
- D4: symbol D_Zener -> back_pcb-rescue:D_Zener
- D5: symbol TL431DBZ -> back_pcb-rescue:TL431DBZ
- J1: symbol Conn_01x12 -> back_pcb-rescue:Conn_01x12
- JP1, JP11, JP12, JP8: symbol JUMPER -> back_pcb-rescue:JUMPER
- L1, L2: symbol L_Small -> back_pcb-rescue:L_Small
- P2, P3: symbol CONN_01X05 -> back_pcb-rescue:CONN_01X05
- P4, P6: symbol CONN_01X06 -> back_pcb-rescue:CONN_01X06
- P7: symbol CONN_01X03 -> back_pcb-rescue:CONN_01X03
- P8: symbol CONN_01X02 -> back_pcb-rescue:CONN_01X02
- P9: symbol USB_A-RESCUE-back_pcb -> back_pcb-rescue:USB_A-RESCUE-back_pcb
- Q1, Q2, Q4, Q5, Q6: symbol Q_PMOS_GSD -> back_pcb-rescue:Q_PMOS_GSD
- Q3: symbol Q_PNP_BEC -> back_pcb-rescue:Q_PNP_BEC
- Q7: symbol BC547 -> back_pcb-rescue:BC547
- R1, R10, R11, R12, R13, R14, R15, R16, R17, R18, R19, R2, R20, R21, R22, R23, R24, R25, R26, R27, R28, R29, R3, R30, R31, R32, R33, R4, R5, R6, R7, R8, R9: symbol R -> back_pcb-rescue:R
- SW1, SW2: symbol SW_PUSH -> back_pcb-rescue:SW_PUSH
- TP1, TP10, TP2, TP3, TP4, TP5, TP6, TP7, TP8, TP9: symbol TEST -> back_pcb-rescue:TEST
- U1: symbol Pi0Top -> pi0outline:Pi0Top
- U2: symbol SIM800_BREAKOUT -> sim800_breakout:SIM800_BREAKOUT
- U3: symbol MCP23017-RESCUE-back_pcb -> back_pcb-rescue:MCP23017-RESCUE-back_pcb
- U4: symbol TP4056_BREAKOUT -> tp4056_breakout:TP4056_BREAKOUT
- U5: symbol 24LC16 -> back_pcb-rescue:24LC16
- U6: symbol DC_DC_BREAKOUT -> dc_dc_breakout:DC_DC_BREAKOUT
- U7: symbol 74LS125 -> back_pcb-rescue:74LS125
- U8: symbol LM339 -> back_pcb-rescue:LM339
- W1, W10, W13, W14, W2, W25, W26, W27, W29, W3, W4, W5, W6, W9: symbol TEST_1P -> back_pcb-rescue:TEST_1P
